File: design-rules/kicad/AISLER-2Layer-Simple/AISLER-2Layer.kicad_pcb (KiCad board)
At the start: 2 copper layers, 0 parts

Commit message: Update KiCad design rules
Other:
- net class Default: via_drill 0.4 -> 0.45
- net class Min: clearance 0.1 -> 0.175; trace_width 0.1 -> 0.2; via_dia 0.7 -> 0.8; via_drill 0.3 -> 0.45
- rule trace_min: 0.1 -> 0.2
- rule via_min_drill: 0.3 -> 0.45
- rule via_min_size: 0.7 -> 0.8
Changed lines of the file:
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@@
-(kicad_pcb (version 20171130) (host pcbnew 5.1.10-88a1d61d58~88~ubuntu20.04.1)
+(kicad_pcb (version 20171130) (host pcbnew "(5.1.10)-1")
   (general
     (thickness 1.6002)
@@
   (setup
     (last_trace_width 0.25)
-    (user_trace_width 0.1)
     (user_trace_width 0.2)
     (user_trace_width 0.5)
@@
     (zone_clearance 0.508)
     (zone_45_only no)
-    (trace_min 0.1)
+    (trace_min 0.2)
     (via_size 0.8)
-    (via_drill 0.4)
-    (via_min_size 0.7)
-    (via_min_drill 0.3)
-    (user_via 0.7 0.3)
-    (user_via 0.8 0.4)
+    (via_drill 0.45)
+    (via_min_size 0.8)
+    (via_min_drill 0.45)
+    (user_via 0.8 0.45)
     (uvia_size 0.8)
-    (uvia_drill 0.4)
+    (uvia_drill 0.45)
     (uvias_allowed no)
     (uvia_min_size 0)
@@
     (solder_mask_min_width 0.1)
     (aux_axis_origin 0 0)
-    (visible_elements FFFFFF7F)
+    (visible_elements 7FFFFFFF)
     (pcbplotparams
       (layerselection 0x010fc_ffffffff)
@@
     (trace_width 0.25)
     (via_dia 0.8)
-    (via_drill 0.4)
+    (via_drill 0.45)
     (uvia_dia 0.8)
-    (uvia_drill 0.4)
+    (uvia_drill 0.45)
     (diff_pair_width 0.25)
     (diff_pair_gap 0.25)
   )
   (net_class Min ""
-    (clearance 0.1)
-    (trace_width 0.1)
-    (via_dia 0.7)
-    (via_drill 0.3)
-    (uvia_dia 0.7)
-    (uvia_drill 0.3)
-    (diff_pair_width 0.12)
-    (diff_pair_gap 0.12)
+    (clearance 0.175)
+    (trace_width 0.2)
+    (via_dia 0.8)
+    (via_drill 0.45)
+    (uvia_dia 0.8)
+    (uvia_drill 0.45)
+    (diff_pair_width 0.25)
+    (diff_pair_gap 0.25)
   )
 )
