File: design-rules/kicad/AISLER-4Layer-Complex/AISLER-4Layer.kicad_pcb (KiCad board)
At the start: 4 copper layers, 0 parts

Commit message: Update KiCad 4 layer design rules
Other:
- net class Min: clearance 0.1 -> 0.125; trace_width 0.1 -> 0.125; via_dia 0.55 -> 0.6
- rule trace_min: 0.1 -> 0.125
- rule via_min_size: 0.55 -> 0.6
Changed lines of the file:
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@@
-(kicad_pcb (version 20171130) (host pcbnew 5.1.10-88a1d61d58~88~ubuntu20.04.1)
+(kicad_pcb (version 20171130) (host pcbnew "(5.1.10)-1")
   (general
     (thickness 1.6)
@@
   (setup
     (last_trace_width 0.25)
-    (user_trace_width 0.1)
-    (user_trace_width 0.25)
+    (user_trace_width 0.125)
     (user_trace_width 0.5)
     (user_trace_width 1)
@@
     (zone_clearance 0.508)
     (zone_45_only no)
-    (trace_min 0.1)
+    (trace_min 0.125)
     (via_size 0.8)
     (via_drill 0.4)
-    (via_min_size 0.55)
+    (via_min_size 0.6)
     (via_min_drill 0.2)
-    (user_via 0.55 0.2)
+    (user_via 0.6 0.2)
     (user_via 1 0.4)
     (uvia_size 0.8)
@@
     (solder_mask_min_width 0.02)
     (aux_axis_origin 0 0)
-    (visible_elements FEFFFF7F)
+    (visible_elements 7FFFFFFF)
     (pcbplotparams
       (layerselection 0x010fc_ffffffff)
@@
   )
   (net_class Min ""
-    (clearance 0.1)
-    (trace_width 0.1)
-    (via_dia 0.55)
+    (clearance 0.125)
+    (trace_width 0.125)
+    (via_dia 0.6)
     (via_drill 0.2)
-    (uvia_dia 0.55)
+    (uvia_dia 0.6)
     (uvia_drill 0.2)
-    (diff_pair_width 0.12)
-    (diff_pair_gap 0.12)
+    (diff_pair_width 0.125)
+    (diff_pair_gap 0.125)
   )
 )
